Commit message: Corrected naming error front_right_calf_link

File: spot_micro_urdf_v2/urdf/spot_micro_urdf_v2.urdf (robot description, URDF)
Before this commit: robot spot_micro_urdf_v2, 13 links, 12 joints
Joints:
- removed joint front_right_calf_link
- added joint front_right_calf_joint: type revolute, parent front_right_thigh_link, child front_right_calf_link, origin xyz=0 -0.118 -0.00045526 rpy=3.14 0 3.14, axis 0 0 1, limit lower=0 upper=3.14 effort=3 velocity=8

Commit message: Updated URDF with correct joint offsets and exra frames for base and feet

File: spot_micro_urdf_v2/urdf/spot_micro_urdf_v2.urdf (robot description, URDF)
Before this commit: robot spot_micro_urdf_v2, 13 links, 12 joints
Links:
- added link LF_FOOT, mass 1e-5; collision cylinder length=0.024 radius=0.012; visual cylinder length=0.024 radius=0.012
- added link LH_FOOT, mass 1e-5; collision cylinder length=0.024 radius=0.012; visual cylinder length=0.024 radius=0.012
- added link RF_FOOT, mass 1e-5; collision cylinder length=0.024 radius=0.012; visual cylinder length=0.024 radius=0.012
- added link RH_FOOT, mass 1e-5; collision cylinder length=0.024 radius=0.012; visual cylinder length=0.024 radius=0.012
- added link base_inertia, mass 0.9248
- link base_link: mass 0.9248 -> None; geometry collision mesh filename=../meshes/base_link.STL; visual mesh filename=../meshes/base_link.STL
- link front_left_calf_link: geometry collision mesh filename=../meshes/front_left_calf_link.STL; visual mesh filename=../meshes/front_left_calf_link.STL
- link front_left_shoulder_link: geometry collision mesh filename=../meshes/front_left_shoulder_link.STL; visual mesh filename=../meshes/front_left_shoulder_link.STL
- link front_left_thigh_link: geometry collision mesh filename=../meshes/front_left_thigh_link.STL; visual mesh filename=../meshes/front_left_thigh_link.STL
- link front_right_calf_link: geometry collision mesh filename=../meshes/front_right_calf_link.STL; visual mesh filename=../meshes/front_right_calf_link.STL
- link front_right_shoulder_link: geometry collision mesh filename=../meshes/front_right_shoulder_link.STL; visual mesh filename=../meshes/front_right_shoulder_link.STL
- link front_right_thigh_link: geometry collision mesh filename=../meshes/front_right_thigh_link.STL; visual mesh filename=../meshes/front_right_thigh_link.STL
- link rear_left_calf_link: geometry collision mesh filename=../meshes/rear_left_calf_link.STL; visual mesh filename=../meshes/rear_left_calf_link.STL
- link rear_left_shoulder_link: geometry collision mesh filename=../meshes/rear_left_shoulder_link.STL; visual mesh filename=../meshes/rear_left_shoulder_link.STL
- link rear_left_thigh_link: geometry collision mesh filename=../meshes/rear_left_thigh_link.STL; visual mesh filename=../meshes/rear_left_thigh_link.STL
- link rear_right_calf_link: geometry collision mesh filename=../meshes/rear_right_calf_link.STL; visual mesh filename=../meshes/rear_right_calf_link.STL
- link rear_right_shoulder_link: geometry collision mesh filename=../meshes/rear_right_shoulder_link.STL; visual mesh filename=../meshes/rear_right_shoulder_link.STL
- link rear_right_thigh_link: geometry collision mesh filename=../meshes/rear_right_thigh_link.STL; visual mesh filename=../meshes/rear_right_thigh_link.STL
Joints:
- added joint FL_lower_leg_2_foot_joint: type fixed, parent front_left_calf_link, child LF_FOOT, origin xyz=-0.011 -0.106 0.023 rpy=0.0 0.0 0.0
- added joint FR_lower_leg_2_foot_joint: type fixed, parent front_right_calf_link, child RF_FOOT, origin xyz=-0.011 -0.106 -0.023 rpy=0.0 0.0 0.0
- added joint RL_lower_leg_2_foot_joint: type fixed, parent rear_left_calf_link, child LH_FOOT, origin xyz=-0.011 -0.106 0.023 rpy=0.0 0.0 0.0
- added joint RR_lower_leg_2_foot_joint: type fixed, parent rear_right_calf_link, child RH_FOOT, origin xyz=-0.011 -0.106 -0.023 rpy=0.0 0.0 0.0
- added joint origin_baselink_joint: type fixed, parent base_link, child base_inertia, origin xyz=0 0 0 rpy=0 0 0
- joint front_left_calf_joint: limit lower=0 upper=3.14 effort=3 velocity=8 -> lower=-2.59 upper=0.1 effort=3 velocity=8
- joint front_left_shoulder_joint: limit lower=0 upper=3.14 effort=3 velocity=8 -> lower=-0.548 upper=0.548 effort=3 velocity=8
- joint front_left_thigh_joint: limit lower=0 upper=3.14 effort=3 velocity=8 -> lower=-2.666 upper=1.548 effort=3 velocity=8; origin xyz=-0.0234 0 0.0226 rpy=0 0 0 -> xyz=-0.0234 0 0.0226 rpy=0 0 0.10521
- joint front_right_calf_joint: limit lower=0 upper=3.14 effort=3 velocity=8 -> lower=-2.59 upper=0.1 effort=3 velocity=8; origin xyz=0 -0.118 -0.00045526 rpy=3.14 0 3.14 -> xyz=0 -0.118 -0.00045526 rpy=3.1378 -0.00040516 3.0364
- joint front_right_shoulder_joint: limit lower=0 upper=3.14 effort=3 velocity=8 -> lower=-0.548 upper=0.548 effort=3 velocity=8
- joint front_right_thigh_joint: limit lower=0 upper=3.14 effort=3 velocity=8 -> lower=-2.666 upper=1.548 effort=3 velocity=8
- joint rear_left_calf_joint: limit lower=0 upper=3.14 effort=3 velocity=8 -> lower=-2.59 upper=0.1 effort=3 velocity=8
- joint rear_left_shoulder_joint: limit lower=0 upper=3.14 effort=3 velocity=8 -> lower=-0.548 upper=0.548 effort=3 velocity=8
- joint rear_left_thigh_joint: limit lower=0 upper=3.14 effort=3 velocity=8 -> lower=-2.666 upper=1.548 effort=3 velocity=8; origin xyz=0.02175 0 0.0226 rpy=0 0 0 -> xyz=0.02175 0 0.0226 rpy=0 0 0.10521
- joint rear_right_calf_joint: limit lower=0 upper=3.14 effort=3 velocity=8 -> lower=-2.59 upper=0.1 effort=3 velocity=8; origin xyz=0 -0.118 -0.00045526 rpy=3.14 0 3.14 -> xyz=0 -0.118 -0.00045526 rpy=3.1378 -0.00040516 3.0364
- joint rear_right_shoulder_joint: limit lower=0 upper=3.14 effort=3 velocity=8 -> lower=-0.548 upper=0.548 effort=3 velocity=8
- joint rear_right_thigh_joint: limit lower=0 upper=3.14 effort=3 velocity=8 -> lower=-2.666 upper=1.548 effort=3 velocity=8
